File: hardware/power_supply.sch (EAGLE design)
At the start: 33 parts, among them Q1 IRF630N, U1 MC34063, U2 AP1507

Commit message: Updating power_supply
Other:
- moved on the sheet: LED1, R7
Changed lines of the file:
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@@
 <parts>
 <part name="U1" library="nixie_ticker" library_urn="urn:adsk.eagle:library:3857935" deviceset="MC34063" device="" package3d_urn="urn:adsk.eagle:package:3949016/1"/>
-<part name="R1" library="resistor" library_urn="urn:adsk.eagle:library:348" deviceset="R-US_" device="R1206" package3d_urn="urn:adsk.eagle:package:26062/1" value="0.5"/>
-<part name="R2" library="resistor" library_urn="urn:adsk.eagle:library:348" deviceset="R-US_" device="R1206" package3d_urn="urn:adsk.eagle:package:26062/1" value="0.5"/>
+<part name="R1" library="resistor" library_urn="urn:adsk.eagle:library:348" deviceset="R-US_" device="R1206" package3d_urn="urn:adsk.eagle:package:23540/2" value="0.5"/>
+<part name="R2" library="resistor" library_urn="urn:adsk.eagle:library:348" deviceset="R-US_" device="R1206" package3d_urn="urn:adsk.eagle:package:23540/2" value="0.5"/>
 <part name="C1" library="nixie_ticker" library_urn="urn:adsk.eagle:library:3857935" deviceset="UUR1C221MCL6GS" device="" package3d_urn="urn:adsk.eagle:package:3945414/1"/>
 <part name="GND1" library="supply1" library_urn="urn:adsk.eagle:library:371" deviceset="GND" device=""/>
@@
 <part name="GND4" library="supply1" library_urn="urn:adsk.eagle:library:371" deviceset="GND" device=""/>
 <part name="GND5" library="supply1" library_urn="urn:adsk.eagle:library:371" deviceset="GND" device=""/>
-<part name="C2" library="resistor" library_urn="urn:adsk.eagle:library:348" deviceset="C-US" device="C0402" package3d_urn="urn:adsk.eagle:package:26136/1"/>
+<part name="C2" library="resistor" library_urn="urn:adsk.eagle:library:348" deviceset="C-US" device="C0402" package3d_urn="urn:adsk.eagle:package:23626/1"/>
 <part name="GND6" library="supply1" library_urn="urn:adsk.eagle:library:371" deviceset="GND" device=""/>
-<part name="C3" library="resistor" library_urn="urn:adsk.eagle:library:348" deviceset="C-US" device="C0402" package3d_urn="urn:adsk.eagle:package:26136/1"/>
+<part name="C3" library="resistor" library_urn="urn:adsk.eagle:library:348" deviceset="C-US" device="C0402" package3d_urn="urn:adsk.eagle:package:23626/1"/>
 <part name="GND7" library="supply1" library_urn="urn:adsk.eagle:library:371" deviceset="GND" device=""/>
 <part name="P+1" library="supply1" library_urn="urn:adsk.eagle:library:371" deviceset="+12V" device=""/>
-<part name="R5" library="resistor" library_urn="urn:adsk.eagle:library:348" deviceset="R-US_" device="R1206" package3d_urn="urn:adsk.eagle:package:26062/1" value="475k"/>
-<part name="R4" library="resistor" library_urn="urn:adsk.eagle:library:348" deviceset="R-US_" device="R1206" package3d_urn="urn:adsk.eagle:package:26062/1" value="13.7k"/>
+<part name="R5" library="resistor" library_urn="urn:adsk.eagle:library:348" deviceset="R-US_" device="R1206" package3d_urn="urn:adsk.eagle:package:23540/2" value="475k"/>
+<part name="R4" library="resistor" library_urn="urn:adsk.eagle:library:348" deviceset="R-US_" device="R1206" package3d_urn="urn:adsk.eagle:package:23540/2" value="13.7k"/>
 <part name="GND8" library="supply1" library_urn="urn:adsk.eagle:library:371" deviceset="GND" device=""/>
-<part name="R6" library="resistor" library_urn="urn:adsk.eagle:library:348" deviceset="R-US_" device="R1206" package3d_urn="urn:adsk.eagle:package:26062/1" value="4.02k"/>
+<part name="R6" library="resistor" library_urn="urn:adsk.eagle:library:348" deviceset="R-US_" device="R1206" package3d_urn="urn:adsk.eagle:package:23540/2" value="4.02k"/>
 <part name="C4" library="nixie_ticker" library_urn="urn:adsk.eagle:library:3857935" deviceset="UUR1C221MCL6GS" device="" package3d_urn="urn:adsk.eagle:package:3945414/1"/>
 <part name="GND9" library="supply1" library_urn="urn:adsk.eagle:library:371" deviceset="GND" device=""/>
@@
 <instance part="C3" gate="G$1" x="55.88" y="10.16"/>
 <instance part="GND7" gate="1" x="55.88" y="2.54"/>
-<instance part="P+1" gate="1" x="-7.62" y="68.58"/>
+<instance part="P+1" gate="1" x="-22.86" y="50.8" rot="R90"/>
 <instance part="R5" gate="G$1" x="63.5" y="27.94" rot="R90"/>
 <instance part="R4" gate="G$1" x="63.5" y="10.16" rot="R90"/>
@@
 <instance part="P+3" gate="1" x="22.86" y="86.36"/>
 <instance part="GND11" gate="1" x="22.86" y="71.12"/>
-<instance part="U$3" gate="G$1" x="-5.08" y="60.96"/>
+<instance part="U$3" gate="G$1" x="-15.24" y="53.34" rot="R90"/>
 <instance part="U$4" gate="G$1" x="101.6" y="35.56" rot="R270"/>
 <instance part="U$5" gate="G$1" x="86.36" y="63.5"/>
@@
 <instance part="+3V1" gate="G$1" x="144.78" y="0" rot="R90"/>
 <instance part="+3V2" gate="G$1" x="114.3" y="2.54" rot="R90"/>
-<instance part="LED1" gate="G$1" x="-17.78" y="43.18"/>
+<instance part="LED1" gate="G$1" x="-10.16" y="48.26"/>
 <instance part="LED2" gate="G$1" x="109.22" y="30.48"/>
-<instance part="R7" gate="G$1" x="-17.78" y="33.02" rot="R90"/>
-<instance part="GND16" gate="1" x="-17.78" y="25.4"/>
+<instance part="R7" gate="G$1" x="-10.16" y="35.56" rot="R90"/>
+<instance part="GND16" gate="1" x="-10.16" y="25.4"/>
 <instance part="R8" gate="G$1" x="109.22" y="20.32" rot="R90"/>
 <instance part="GND17" gate="1" x="109.22" y="12.7"/>
@@
 <pinref part="C1" gate="G$1" pin="-"/>
 <pinref part="GND1" gate="1" pin="GND"/>
+<wire x1="35.56" y1="45.72" x2="35.56" y2="43.18" width="0.1524" layer="91"/>
 </segment>
 <segment>
@@
 <pinref part="GND9" gate="1" pin="GND"/>
 <pinref part="C4" gate="G$1" pin="-"/>
-<wire x1="71.12" y1="27.94" x2="71.12" y2="30.48" width="0.1524" layer="91"/>
 </segment>
 <segment>
@@
 <wire x1="22.86" y1="78.74" x2="22.86" y2="76.2" width="0.1524" layer="91"/>
 <pinref part="C5" gate="G$1" pin="-"/>
-<wire x1="22.86" y1="76.2" x2="30.48" y2="76.2" width="0.1524" layer="91"/>
+<wire x1="22.86" y1="76.2" x2="30.48" y2="73.66" width="0.1524" layer="91"/>
 </segment>
 <segment>
@@
 <pinref part="C6" gate="G$1" pin="-"/>
 <wire x1="137.16" y1="25.4" x2="149.86" y2="25.4" width="0.1524" layer="91"/>
-<wire x1="149.86" y1="25.4" x2="149.86" y2="27.94" width="0.1524" layer="91"/>
 </segment>
 <segment>
@@
 <pinref part="R7" gate="G$1" pin="1"/>
 <pinref part="GND16" gate="1" pin="GND"/>
+<wire x1="-10.16" y1="30.48" x2="-10.16" y2="27.94" width="0.1524" layer="91"/>
 </segment>
 <segment>
@@
 <wire x1="-5.08" y1="45.72" x2="-2.54" y2="45.72" width="0.1524" layer="91"/>
 <pinref part="R1" gate="G$1" pin="1"/>
-<wire x1="-5.08" y1="45.72" x2="-5.08" y2="50.8" width="0.1524" layer="91"/>
-<wire x1="-5.08" y1="50.8" x2="-5.08" y2="53.34" width="0.1524" layer="91"/>
+<wire x1="-5.08" y1="45.72" x2="-5.08" y2="53.34" width="0.1524" layer="91"/>
 <wire x1="-5.08" y1="53.34" x2="-2.54" y2="53.34" width="0.1524" layer="91"/>
-<wire x1="-5.08" y1="55.88" x2="-5.08" y2="53.34" width="0.1524" layer="91"/>
 <pinref part="U$3" gate="G$1" pin="2"/>
 <pinref part="LED1" gate="G$1" pin="A"/>
-<wire x1="-17.78" y1="45.72" x2="-17.78" y2="50.8" width="0.1524" layer="91"/>
-<wire x1="-17.78" y1="50.8" x2="-5.08" y2="50.8" width="0.1524" layer="91"/>
+<wire x1="-10.16" y1="53.34" x2="-5.08" y2="53.34" width="0.1524" layer="91"/>
+<wire x1="-10.16" y1="50.8" x2="-10.16" y2="53.34" width="0.1524" layer="91"/>
 </segment>
 </net>
@@
 <pinref part="LED1" gate="G$1" pin="C"/>
 <pinref part="R7" gate="G$1" pin="2"/>
-</segment>
-</net>
+<wire x1="-10.16" y1="43.18" x2="-10.16" y2="40.64" width="0.1524" layer="91"/>
+</segment>
+</net>

Commit message: Updating 8-12
Parts:
- removed JP1: (no value), pinhead:PINHD-1X6
- removed U$2: 3309P-1-202, nixie_ticker:3309P-1-202
- removed U$4: T411001B, nixie_ticker:T411001B
- added C7, C8: (no value), resistor:C-USC0402
- added F1, F2: FUSE_1206, nixie_ticker:FUSE_1206
- added JP3: (no value), pinhead:PINHD-1X5
- added RX: 2k, nixie_ticker:3309P-1-202
- added SW2: T411001B, nixie_ticker:T411001B
- added U3: CD40109B_SPLITEN, nixie_ticker:CD40109B_SPLITEN
- C1, C5, C6: value UUR1C221MCL6GS -> 220uF
- C2: value (none) -> 680pF
- C3: value (none) -> 0.01uF
- C4: value UUR1C221MCL6GS -> 3.3uF
- L1: value RLB9012 -> 100uH
- R3: device resistor:R-US_R0402 -> resistor:R-US_R0805
- R7, R8: value 1k -> 2k; device resistor:R-US_R0402 -> resistor:R-US_R0805
- renumbered LED1 to HV, LED2 to LOGIC, U$3 to SW1, U$9 to L2
Connections:
- removed net DI: JP1.6, JP2.2
- removed net SHCP: JP1.5, JP2.1
- removed net STCP: JP1.4, JP2.3
- new net CLK_H: JP3.4, U3.G
- new net CLK_L: JP2.1, U3.C
- new net DATA_H: JP3.5, U3.F
- new net DATA_L: JP2.2, U3.D
- new net LATCH_H: JP3.3, U3.H
- new net LATCH_L: JP2.3, U3.B
- new net N$13: F1.2, SW2.2, SW2.3
- new net N$14: F2.2, SW1.1
- net +12V: now also F1.1, F2.1; no longer SW1.1, U$4.2
- net +3V3: now also C7.1, U3.EN_B, U3.EN_C, U3.EN_D, U3.VCC; no longer JP1.3
- net +5V: now also C8.1, JP3.2, U3.VDD; no longer JP1.2
- net GND: now also C7.2, C8.2, JP3.1, RX.P$3, U3.A, U3.E, U3.EN_A, U3.VSS; no longer JP1.1, U$2.P$3
- net N$3: now also RX.P$2; no longer U$2.P$2
- net N$8: now also SW2.1; no longer U$4.1
Other:
- moved on the sheet: C3, C5

Commit message: Final update before submitting to PCB shop
Parts:
- RX: device nixie_ticker:3309P-1-202 -> nixie_ticker:TC33X-2
- U2: value AP1507 -> AP1507SOIC-8; device nixie_ticker:AP1507 -> nixie_ticker:AP1507SOIC-8
Changed lines of the file:
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@@
 <part name="GND2" library="supply1" library_urn="urn:adsk.eagle:library:371" deviceset="GND" device=""/>
 <part name="D2" library="nixie_ticker" library_urn="urn:adsk.eagle:library:3857935" deviceset="MMBD914L" device="" package3d_urn="urn:adsk.eagle:package:43389/2" value=""/>
-<part name="Q2" library="transistor" library_urn="urn:adsk.eagle:library:402" deviceset="*-PNP-" device="SOT23-BEC" package3d_urn="urn:adsk.eagle:package:29919/2" technology="BC807-16"/>
+<part name="Q2" library="transistor" library_urn="urn:adsk.eagle:library:402" deviceset="*-PNP-" device="SOT23-BEC" package3d_urn="urn:adsk.eagle:package:28748/2" technology="BC807-16"/>
 <part name="R3" library="resistor" library_urn="urn:adsk.eagle:library:348" deviceset="R-US_" device="R0805" package3d_urn="urn:adsk.eagle:package:23553/2" value="1k"/>
 <part name="GND3" library="supply1" library_urn="urn:adsk.eagle:library:371" deviceset="GND" device=""/>
@@
 <part name="GND9" library="supply1" library_urn="urn:adsk.eagle:library:371" deviceset="GND" device=""/>
 <part name="P+2" library="supply1" library_urn="urn:adsk.eagle:library:371" deviceset="V+" device=""/>
-<part name="RX" library="nixie_ticker" library_urn="urn:adsk.eagle:library:3857935" deviceset="3309P-1-202" device="" package3d_urn="urn:adsk.eagle:package:3997919/2" value="2k"/>
+<part name="RX" library="nixie_ticker" library_urn="urn:adsk.eagle:library:3857935" deviceset="TC33X-2" device="" package3d_urn="urn:adsk.eagle:package:4765398/2" value="2k"/>
 <part name="GND10" library="supply1" library_urn="urn:adsk.eagle:library:371" deviceset="GND" device=""/>
 <part name="U$1" library="nixie_ticker" library_urn="urn:adsk.eagle:library:3857935" deviceset="EJ508A" device="" package3d_urn="urn:adsk.eagle:package:3997947/2"/>
@@
 <part name="P+4" library="supply1" library_urn="urn:adsk.eagle:library:371" deviceset="V+" device=""/>
 <part name="GND12" library="supply1" library_urn="urn:adsk.eagle:library:371" deviceset="GND" device=""/>
-<part name="U2" library="nixie_ticker" library_urn="urn:adsk.eagle:library:3857935" deviceset="AP1507" device="" package3d_urn="urn:adsk.eagle:package:4010820/1"/>
+<part name="U2" library="nixie_ticker" library_urn="urn:adsk.eagle:library:3857935" deviceset="AP1507" device="SOIC-8" package3d_urn="urn:adsk.eagle:package:3949016/1" value="AP1507SOIC-8"/>
 <part name="P+5" library="supply1" library_urn="urn:adsk.eagle:library:371" deviceset="+12V" device=""/>
 <part name="C5" library="nixie_ticker" library_urn="urn:adsk.eagle:library:3857935" deviceset="UUR1C221MCL6GS" device="" package3d_urn="urn:adsk.eagle:package:3945414/1" value="220uF"/>

Commit message: Updates 8-28
Parts:
- C2, C3: device resistor:C-USC0402 -> nixie_ticker:C0402
- C7, C8: value (none) -> 1uF; device resistor:C-USC0402 -> nixie_ticker:C0402
- HV, LOGIC: device led:LEDSML0805 -> led:LEDCHIP-LED0805
Connections:
- net +3V3: now also C7.+; no longer C7.1
- net +5V: now also C8.+; no longer C8.1
- net GND: now also C2.-, C3.-, C7.-, C8.-; no longer C2.2, C3.2, C7.2, C8.2
- net N$7: now also C2.+; no longer C2.1
- net N$9: now also C3.+; no longer C3.1
Changed lines of the file:
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@@
 <part name="GND3" library="supply1" library_urn="urn:adsk.eagle:library:371" deviceset="GND" device=""/>
 <part name="GND4" library="supply1" library_urn="urn:adsk.eagle:library:371" deviceset="GND" device=""/>
-<part name="C2" library="resistor" library_urn="urn:adsk.eagle:library:348" deviceset="C-US" device="C0402" package3d_urn="urn:adsk.eagle:package:23626/1" value="680pF"/>
-<part name="C3" library="resistor" library_urn="urn:adsk.eagle:library:348" deviceset="C-US" device="C0402" package3d_urn="urn:adsk.eagle:package:23626/1" value="0.01uF"/>
+<part name="C2" library="nixie_ticker" library_urn="urn:adsk.eagle:library:3857935" deviceset="C0402" device="" package3d_urn="urn:adsk.eagle:package:4771247/2" value="680pF"/>
+<part name="C3" library="nixie_ticker" library_urn="urn:adsk.eagle:library:3857935" deviceset="C0402" device="" package3d_urn="urn:adsk.eagle:package:4771247/2" value="0.01uF"/>
 <part name="GND7" library="supply1" library_urn="urn:adsk.eagle:library:371" deviceset="GND" device=""/>
 <part name="P+1" library="supply1" library_urn="urn:adsk.eagle:library:371" deviceset="+12V" device=""/>
@@
 <part name="GND15" library="supply1" library_urn="urn:adsk.eagle:library:371" deviceset="GND" device=""/>
 <part name="+3V1" library="supply1" library_urn="urn:adsk.eagle:library:371" deviceset="+3V3" device=""/>
-<part name="HV" library="led" library_urn="urn:adsk.eagle:library:259" deviceset="LED" device="SML0805" package3d_urn="urn:adsk.eagle:package:15830/1"/>
-<part name="LOGIC" library="led" library_urn="urn:adsk.eagle:library:259" deviceset="LED" device="SML0805" package3d_urn="urn:adsk.eagle:package:15830/1"/>
+<part name="HV" library="led" library_urn="urn:adsk.eagle:library:259" deviceset="LED" device="CHIP-LED0805" package3d_urn="urn:adsk.eagle:package:15818/2"/>
+<part name="LOGIC" library="led" library_urn="urn:adsk.eagle:library:259" deviceset="LED" device="CHIP-LED0805" package3d_urn="urn:adsk.eagle:package:15818/2"/>
 <part name="R7" library="resistor" library_urn="urn:adsk.eagle:library:348" deviceset="R-US_" device="R0805" package3d_urn="urn:adsk.eagle:package:23553/2" value="2k"/>
 <part name="GND16" library="supply1" library_urn="urn:adsk.eagle:library:371" deviceset="GND" device=""/>
@@
 <part name="GND18" library="supply1" library_urn="urn:adsk.eagle:library:371" deviceset="GND" device=""/>
 <part name="P+9" library="supply1" library_urn="urn:adsk.eagle:library:371" deviceset="+5V" device=""/>
-<part name="C7" library="resistor" library_urn="urn:adsk.eagle:library:348" deviceset="C-US" device="C0402" package3d_urn="urn:adsk.eagle:package:23626/1"/>
-<part name="C8" library="resistor" library_urn="urn:adsk.eagle:library:348" deviceset="C-US" device="C0402" package3d_urn="urn:adsk.eagle:package:23626/1"/>
+<part name="C7" library="nixie_ticker" library_urn="urn:adsk.eagle:library:3857935" deviceset="C0402" device="" package3d_urn="urn:adsk.eagle:package:4771247/2" value="1uF"/>
+<part name="C8" library="nixie_ticker" library_urn="urn:adsk.eagle:library:3857935" deviceset="C0402" device="" package3d_urn="urn:adsk.eagle:package:4771247/2" value="1uF"/>
 <part name="GND14" library="supply1" library_urn="urn:adsk.eagle:library:371" deviceset="GND" device=""/>
 <part name="GND20" library="supply1" library_urn="urn:adsk.eagle:library:371" deviceset="GND" device=""/>
@@
 </segment>
 <segment>
-<pinref part="C3" gate="G$1" pin="2"/>
+<pinref part="C3" gate="G$1" pin="-"/>
 <pinref part="GND7" gate="1" pin="GND"/>
 </segment>
@@
 <pinref part="GND16" gate="1" pin="GND"/>
 <wire x1="-10.16" y1="30.48" x2="-10.16" y2="12.7" width="0.1524" layer="91"/>
-<pinref part="C2" gate="G$1" pin="2"/>
+<pinref part="C2" gate="G$1" pin="-"/>
 <wire x1="-5.08" y1="15.24" x2="-5.08" y2="12.7" width="0.1524" layer="91"/>
 <wire x1="-10.16" y1="12.7" x2="-5.08" y2="12.7" width="0.1524" layer="91"/>
@@
 </segment>
 <segment>
-<pinref part="C7" gate="G$1" pin="2"/>
+<pinref part="C7" gate="G$1" pin="-"/>
 <pinref part="GND14" gate="1" pin="GND"/>
 </segment>
 <segment>
-<pinref part="C8" gate="G$1" pin="2"/>
+<pinref part="C8" gate="G$1" pin="-"/>
 <pinref part="GND20" gate="1" pin="GND"/>
 </segment>
@@
 <pinref part="U1" gate="G$1" pin="CT"/>
 <wire x1="2.54" y1="27.94" x2="-5.08" y2="27.94" width="0.1524" layer="91"/>
-<pinref part="C2" gate="G$1" pin="1"/>
+<pinref part="C2" gate="G$1" pin="+"/>
 <wire x1="-5.08" y1="27.94" x2="-5.08" y2="22.86" width="0.1524" layer="91"/>
 </segment>
@@
 <wire x1="17.78" y1="17.78" x2="17.78" y2="0" width="0.1524" layer="91"/>
 <wire x1="17.78" y1="0" x2="48.26" y2="0" width="0.1524" layer="91"/>
-<pinref part="C3" gate="G$1" pin="1"/>
+<pinref part="C3" gate="G$1" pin="+"/>
 <wire x1="48.26" y1="0" x2="48.26" y2="15.24" width="0.1524" layer="91"/>
 <wire x1="48.26" y1="15.24" x2="63.5" y2="15.24" width="0.1524" layer="91"/>
@@
 <pinref part="U3" gate="G$1" pin="VDD"/>
 <pinref part="P+7" gate="1" pin="+5V"/>
-<pinref part="C8" gate="G$1" pin="1"/>
+<pinref part="C8" gate="G$1" pin="+"/>
 <wire x1="154.94" y1="-17.78" x2="160.02" y2="-17.78" width="0.1524" layer="91"/>
 <wire x1="160.02" y1="-17.78" x2="160.02" y2="-12.7" width="0.1524" layer="91"/>
@@
 </segment>
 <segment>
-<pinref part="C7" gate="G$1" pin="1"/>
+<pinref part="C7" gate="G$1" pin="+"/>
 <pinref part="U3" gate="G$1" pin="VCC"/>
 <pinref part="+3V2" gate="G$1" pin="+3V3"/>
